File: memento.kicad_pcb (KiCad board)
At the start: 2 copper layers, 150 x 100 mm, 6 parts, among them U1 XIAO_ESP32C3

Commit message: pcb updated
Parts:
- removed D1: LED, LED_0805_2012Metric
- removed kibuzzard-6AB60A4F: G***, kibuzzard-6AB60A4F
- added D2: WS2812B, memento:WS2812B_PLCC4_5.0x5.0mm, F.Cu at (187.3, 74.0)
- added D3: WS2812B, memento:WS2812B_PLCC4_5.0x5.0mm, F.Cu at (166.2, 45.4)
- added D4: WS2812B, memento:WS2812B_PLCC4_5.0x5.0mm, F.Cu at (144.3, 73.3)
- added D5: WS2812B, memento:WS2812B_PLCC4_5.0x5.0mm, F.Cu at (166.2, 96.4)
- added kibuzzard-6AB62C58: G***, kibuzzard-6AB62C58, F.Cu at (165.0, 133.6)
- added kibuzzard-6AB62C70: G***, kibuzzard-6AB62C70, F.Cu at (227.6, 64.9)
- R1: footprint R_0805_2012Metric -> Resistor_SMD:R_0805_2012Metric
- U1: footprint XIAO-ESP32C3-Hybrid -> memento:XIAO-ESP32C3-Hybrid
- moved U1 20.4 mm to (228.4, 89.2)
- moved R1 15.0 mm to (232.5, 75.4)
- moved LOGO2 7.97 mm to (164.9, 109.2)
- moved LOGO1 1.80 mm to (164.9, 71.4)
Connections:
- R1 pad 2: unconnected-(R1-Pad2) -> Net-(U1-D0/A0)
- U1 pad 1: unconnected-(U1-D0/A0-Pad1) -> Net-(U1-D0/A0)
- U1 pad 13: unconnected-(U1-GND-Pad13) -> GND
- U1 pad 14: unconnected-(U1-5V-Pad14) -> +5V

Commit message: routing updated
Parts:
- added U2: BMP280_Module, memento:BMP280_Module_GY_6P_15x11.5mm, B.Cu at (104.9, 86.8)
- moved kibuzzard-6AB62C70 114.0 mm to (115.5, 44.3)
- moved kibuzzard-6AB62C58 100.1 mm to (210.8, 44.6)
- moved R1 39.4 mm to (193.8, 83.0), turned to -90 degrees
- moved D5 9.47 mm to (164.7, 105.8), turned to 180 degrees
- moved D2 9.01 mm to (187.3, 83.0)
- moved D3 9.01 mm to (166.1, 54.4)
- moved D4 9.01 mm to (144.3, 82.4)
- moved LOGO1 9.01 mm to (164.9, 80.4)
- moved LOGO2 9.01 mm to (164.9, 118.2)
Connections:
- U1 pad 5: unconnected-(U1-D4/SDA-Pad5) -> Net-(U1-D4/SDA)
- U1 pad 6: unconnected-(U1-D5/SCL-Pad6) -> Net-(U1-D5/SCL)
Routing:
- net GND: track 0.00 -> 291.3 mm
- net +5V: track 0.00 -> 230.3 mm
- net Net-(U1-D4/SDA): track 0.00 -> 181.4 mm
- net Net-(U1-D5/SCL): track 0.00 -> 173.0 mm
- net Net-(D2-DOUT): track 0.00 -> 49.9 mm
- net Net-(U1-D0/A0): track 0.00 -> 44.0 mm
- net Net-(D4-DOUT): track 0.00 -> 42.0 mm
- net Net-(D3-DOUT): track 0.00 -> 39.7 mm
- net Net-(D2-DIN): track 0.00 -> 4.40 mm
Other:
- outline, holes or cut-outs redrawn
