File: memento.kicad_sch (KiCad schematic)
At the start: 3 parts, among them U1 XIAO_ESP32C3

Commit message: pcb updated
Parts:
- removed D1: LED, LED_SMD:LED_0805_2012Metric, symbol Device:LED
- added D2, D3, D4, D5: WS2812B, memento:WS2812B_PLCC4_5.0x5.0mm, symbol memento:WS2812B
- R1: footprint Resistor_SMD:R_0805_2012Metric -> (none)
Connections:
- net at U1.1 (D0/A0): now also R1.2
- net GND: now reaches U1.13 (GND)
- net GND: now also D2.3 (VSS), D3.3 (VSS), D4.3 (VSS), D5.3 (VSS)
- net +5V: now reaches U1.14 (5V)
- net +5V: now also D2.1 (VDD), D3.1 (VDD), D4.1 (VDD), D5.1 (VDD)
- net at R1.1: now also D2.4 (DIN)
- new net: D2.2 (DOUT), D3.4 (DIN)
- new net: D4.2 (DOUT), D5.4 (DIN)
- new net: D3.2 (DOUT), D4.4 (DIN)

Commit message: routing updated
Parts:
- added U2: BMP280_Module, memento:BMP280_Module_GY_6P_15x11.5mm, symbol memento:BMP280_Module
Connections:
- net +5V: now also U2.1 (VCC)
- net GND: now also U2.2 (GND)
- net at U1.5 (D4/SDA): now also U2.4 (SDA)
- net at U1.6 (D5/SCL): now also U2.3 (SCL)
Other:
- moved on the sheet: D2, D3, D4, D5, R1, U1
