File: hw/memento.kicad_pcb (KiCad board)
At the start: 2 copper layers, 150 x 100 mm, 11 parts, among them U1 XIAO_ESP32C3, U2 BMP280_Module

Commit message: files updated
Parts:
- added R2: R_US, Resistor_SMD:R_0805_2012Metric, F.Cu at (109.2, 92.2)
- added R3: R_US, Resistor_SMD:R_0805_2012Metric, F.Cu at (100.8, 92.3)
- moved kibuzzard-6AB62C70 1.72 mm to (116.9, 43.3)
- moved kibuzzard-6AB62C58 1.04 mm to (210.8, 43.6)
Connections:
- U1 pad 12: unconnected-(U1-3V3-Pad12) -> +3.3V
- U2 pad 1: +5V -> +3.3V
Routing:
- net +3.3V: track 0.00 -> 210.7 mm, vias 0 -> 2
- net +5V: track 230.3 -> 194.9 mm
- net GND: track 291.3 -> 280.3 mm
- net Net-(U1-D5/SCL): track 173.0 -> 180.1 mm
- net Net-(U1-D4/SDA): track 181.4 -> 188.3 mm
