File: hw/memento.kicad_sch (KiCad schematic)
At the start: 7 parts, among them U1 XIAO_ESP32C3, U2 BMP280_Module

Commit message: files updated
Parts:
- added R2, R3: R_US, Resistor_SMD:R_0805_2012Metric, symbol Device:R_US
- R1: footprint (none) -> Resistor_SMD:R_0805_2012Metric
Connections:
- net +5V: no longer U2.1 (VCC)
- net +3.3V: now reaches U1.12 (3V3)
- net +3.3V: now also U2.1 (VCC), R2.2, R3.2
- net at U1.5 (D4/SDA), U2.4 (SDA): now also R3.1
- net at U1.6 (D5/SCL), U2.3 (SCL): now also R2.1
